File: DRV8213 brushed Motor Driver.kicad_pcb (KiCad board)
At the start: 4 copper layers, 15 x 15 mm, 26 parts, among them J1 Keystone 6102, J10 Precidip 852-10-004-20-001101, J11 Precidip 852-10-004-20-001101, J2 Keystone 6102, J3 Keystone 6100, J4 Keystone 6100, J5 Keystone 6102, J6 Keystone 6102, J7 Keystone 6100, J8 Keystone 6100, J9 JST PH 2mm horizontal, U1 DRV8213RTER, U2 LP2981-3.3

Commit message: Fixed critical error
Parts:
- moved C5 0.10 mm to (171.4, 108.5)
Routing:
- net VDD: vias 14 -> 21
- net GNDPWR: vias 28 -> 34
Changed lines of the file:
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@@
 	(footprint "Capacitor_SMD:C_0603_1608Metric"
 		(layer "F.Cu")
-		(at 171.475 108.525 180)
+		(at 171.375 108.525 180)
 		(descr "Capacitor SMD 0603 (1608 Metric), square (rectangular) end terminal, IPC_7351 nominal, (Body size source: IPC-SM-782 page 76, https://www.pcb-3d.com/wordpress/wp-content/uploads/ipc-sm-782a_amendment_1_and_2.pdf), generated with kicad-footprint-generator")
 		(tags "capacitor")
@@
 	)
 	(via
+		(at 178.3 107.675)
+		(size 0.6)
+		(drill 0.3)
+		(layers "F.Cu" "B.Cu")
+		(free yes)
+		(net 1)
+	)
+	(via
+		(at 178.225 96.475)
+		(size 0.6)
+		(drill 0.3)
+		(layers "F.Cu" "B.Cu")
+		(free yes)
+		(net 1)
+	)
+	(via
 		(at 177.475 104.55)
 		(size 0.6)
@@
 	)
 	(via
+		(at 178.25 98.175)
+		(size 0.6)
+		(drill 0.3)
+		(layers "F.Cu" "B.Cu")
+		(free yes)
+		(net 1)
+	)
+	(via
 		(at 178.3 105.05)
 		(size 0.6)
@@
 	)
 	(via
+		(at 178.275 106)
+		(size 0.6)
+		(drill 0.3)
+		(layers "F.Cu" "B.Cu")
+		(free yes)
+		(net 1)
+	)
+	(via
 		(at 178.275 99.95)
 		(size 0.6)
@@
 	)
 	(via
+		(at 178.3 106.825)
+		(size 0.6)
+		(drill 0.3)
+		(layers "F.Cu" "B.Cu")
+		(free yes)
+		(net 1)
+	)
+	(via
+		(at 178.225 95.65)
+		(size 0.6)
+		(drill 0.3)
+		(layers "F.Cu" "B.Cu")
+		(free yes)
+		(net 1)
+	)
+	(via
 		(at 178.275 101.7)
 		(size 0.6)
@@
 		(net 1)
 	)
+	(via
+		(at 178.225 97.3)
+		(size 0.6)
+		(drill 0.3)
+		(layers "F.Cu" "B.Cu")
+		(free yes)
+		(net 1)
+	)
 	(segment
 		(start 165.5 101.7)
@@
 	)
 	(via
+		(at 169.6 108.55)
+		(size 0.6)
+		(drill 0.3)
+		(layers "F.Cu" "B.Cu")
+		(free yes)
+		(net 2)
+	)
+	(via
 		(at 166 105.05)
 		(size 0.6)
@@
 	)
 	(via
+		(at 168 108.55)
+		(size 0.6)
+		(drill 0.3)
+		(layers "F.Cu" "B.Cu")
+		(free yes)
+		(net 2)
+	)
+	(via
+		(at 168.8 108.55)
+		(size 0.6)
+		(drill 0.3)
+		(layers "F.Cu" "B.Cu")
+		(free yes)
+		(net 2)
+	)
+	(via
 		(at 173.45 98.6)
 		(size 0.6)
@@
 	)
 	(via
+		(at 168 107.75)
+		(size 0.6)
+		(drill 0.3)
+		(layers "F.Cu" "B.Cu")
+		(free yes)
+		(net 2)
+	)
+	(via
 		(at 173.45 99.4)
 		(size 0.6)
@@
 	)
 	(via
+		(at 168.8 107.75)
+		(size 0.6)
+		(drill 0.3)
+		(layers "F.Cu" "B.Cu")
+		(free yes)
+		(net 2)
+	)
+	(via
 		(at 164.425 95.825)
 		(size 0.6)
@@
 		(net 2)
 	)
+	(via
+		(at 169.6 107.75)
+		(size 0.6)
+		(drill 0.3)
+		(layers "F.Cu" "B.Cu")
+		(free yes)
+		(net 2)
+	)
 	(segment
 		(start 173.5 100.8)
@@
 		(polygon
 			(pts
-				(xy 176.6 98.675) (xy 177.5 98.675) (xy 178.8 98.6) (xy 178.8 105.6) (xy 178.125 105.675) (xy 177.225 105.675)
-				(xy 176.6 104.125)
+				(xy 176.6 98.675) (xy 177.8 98.245) (xy 177.775 95.225) (xy 178.8 95.225) (xy 178.8 108.2) (xy 177.875 108.2)
+				(xy 177.6 106.7) (xy 177.225 105.675) (xy 176.6 104.125)
 			)
 		)
